Commit message: added manual gripper example setup

File: hippo_sim/models/gripper/urdf/gripper.urdf (robot description, URDF)
Before this commit: robot hippocampus, 8 links, 7 joints
Links:
- removed link base_link
- removed link left_jaw
- removed link left_prismatic_link
- removed link left_prismatic_revolute_link
- removed link left_rotation_dummy_link
- removed link left_rotation_link
- removed link prismatic_link
- added link end_effector_base_link, mass 0.1; visual mesh filename=file:///home/ros-user/uuv/ros2/install/hippo_sim/share/hipp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
- added link end_effector_left_inner_revolute_link, mass 0.1; visual cylinder length=0.005 radius=0.01
- added link end_effector_left_jaw_link, mass 0.1; visual mesh filename=file:///home/ros-user/uuv/ros2/install/hippo_sim/share/hipp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
- added link end_effector_left_prismatic_link, mass 0.1
- added link end_effector_left_revolute_link, mass 0.1; visual cylinder length=0.02 radius=0.0025
- added link end_effector_prismatic_link, mass 0.1; visual cylinder length=0.02 radius=0.0025
- added link end_effector_right_inner_revolute_link, mass 0.1; visual cylinder length=0.005 radius=0.01
- added link end_effector_right_jaw_link, mass 0.1; visual mesh filename=file:///home/ros-user/uuv/ros2/install/hippo_sim/share/hipp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
- added link end_effector_right_prismatic_link, mass 0.1
- added link end_effector_right_revolute_link, mass 0.1; visual cylinder length=0.02 radius=0.0025
Joints:
- removed joint dummy_joint
- removed joint left_jaw_joint
- removed joint left_prismatic_joint
- removed joint left_prismatic_revolute_joint
- removed joint left_revolute_joint
- removed joint prismatic_joint
- added joint end_effector_left_inner_revolute_joint: type continuous, parent end_effector_prismatic_link, child end_effector_left_inner_revolute_link, axis 0 0 1
- added joint end_effector_left_jaw_joint: type fixed, parent end_effector_left_prismatic_link, child end_effector_left_jaw_link, origin xyz=0 8.5e-3 0
- added joint end_effector_left_prismatic_joint: type prismatic, parent end_effector_left_inner_revolute_link, child end_effector_left_prismatic_link, origin xyz=0 7.0e-3 0, axis 0 1 0, limit lower=-1.0 upper=1.0 effort=100 velocity=1.0
- added joint end_effector_left_revolute_joint: type continuous, parent end_effector_left_jaw_link, child end_effector_left_revolute_link, axis 0 0 1
- added joint end_effector_right_inner_revolute_joint: type continuous, parent end_effector_prismatic_link, child end_effector_right_inner_revolute_link, axis 0 0 1
- added joint end_effector_right_jaw_joint: type fixed, parent end_effector_right_prismatic_link, child end_effector_right_jaw_link, origin xyz=0 -8.5e-3 0
- added joint end_effector_right_prismatic_joint: type prismatic, parent end_effector_right_inner_revolute_link, child end_effector_right_prismatic_link, origin xyz=0 -7.0e-3 0, axis 0 1 0, limit lower=-1.0 upper=1.0 effort=100 velocity=1.0
- added joint end_effector_right_revolute_joint: type continuous, parent end_effector_right_jaw_link, child end_effector_right_revolute_link, axis 0 0 1
- added joint joint_5: type prismatic, parent end_effector_base_link, child end_effector_prismatic_link, origin xyz=6.9e-3 0 0, axis 1 0 0, limit lower=0.0 upper=0.012 effort=28.992 velocity=2.0
- joint attachment: child base_link -> end_effector_base_link

File: hippo_sim/models/gripper/urdf/gripper.xacro (robot description, xacro)
@@ -1,4 +1,8 @@
 <?xml version="1.0"?>
 <robot xmlns:xacro="http://www.ros.org/wiki/xacro" name="hippocampus">
+    <xacro:include filename="$(find hippo_sim)/models/gripper/urdf/alpha_end_effector.xacro" />
+    <link name="world" />
+    <xacro:end_effector prefix="end_effector" parent="world" />
+    <!--
     <xacro:include filename="$(find hippo_sim)/models/common/urdf/common.xacro" />
     <xacro:macro name="dummy_inertia">
@@ -22,11 +26,4 @@
         </visual>
     </link>
-    <!--
-    <joint name="left_fixed_joint" type="fixed">
-        <parent link="base_link" />
-        <origin xyz="1 1 0" rpy="0 0 0" />
-        <child link="left_rotation_link" />
-    </joint>
-    -->
     <link name="prismatic_link">
         <xacro:dummy_inertia />
@@ -145,3 +142,4 @@
         </plugin>
     </gazebo>
+    -->
 </robot>
